File: 368255-2.kicad_sch (KiCad schematic)
At the start: 25 parts, among them J10 5569-16A2, J2 5569-20A2, J21 Conn_01x01_Pin, J22 Conn_01x01_Pin, J23 Conn_01x01_Pin, J24 Conn_01x01_Pin, J25 Conn_01x01_Pin, J26 Conn_01x01_Pin, J27 Conn_01x01_Pin, J28 Conn_01x01_Pin, J3 5569-06A2, J4 5569-08A2, J5 5569-18A2, P1 368255-2, U1 ULN2003A

Commit message: removed unnececary silk+nets+title frame
Parts:
- removed R5, R6, R7: 10k, Resistor_SMD:R_0201_0603Metric, symbol Device:R
Other:
- company: DAECU -> wmrk
- title: ECU adapter -> ECU uaefi to 368255-2 adapter
